Commit message: se ajusta el codigo para solo tenga una articulacion

File: src/test1_ros2control/description/ros2_control/rrbot.ros2_control.xacro (robot description, xacro)
@@ -16,5 +16,5 @@
         <state_interface name="position"/>
       </joint>
-      <joint name="${prefix}joint2">
+      <!-- <joint name="${prefix}joint2">
         <command_interface name="position">
           <param name="min">-1</param>
@@ -22,5 +22,5 @@
         </command_interface>
         <state_interface name="position"/>
-      </joint>
+      </joint> -->
     </ros2_control>
   </xacro:macro>

File: src/test1_ros2control/description/urdf/rrbot_description.urdf.xacro (robot description, xacro)
@@ -7,5 +7,5 @@
   <xacro:property name="height1" value="2" /> <!-- Link 1 -->
   <xacro:property name="height2" value="1" /> <!-- Link 2 -->
-  <xacro:property name="height3" value="1" /> <!-- Link 3 -->
+  <!-- <xacro:property name="height3" value="1" /> Link 3 -->
   <xacro:property name="axel_offset" value="0.05" /> <!-- Space btw top of beam and the each joint -->
   <joint name="${prefix}base_joint" type="fixed">
@@ -70,5 +70,5 @@
     </inertial>
   </link>
-  <joint name="${prefix}joint2" type="continuous">
+  <!-- <joint name="${prefix}joint2" type="continuous">
     <parent link="${prefix}link1"/>
     <child link="${prefix}link2"/>
@@ -77,7 +77,7 @@
     <dynamics damping="0.7"/>
     <limit effort="100" velocity="1.0"/>
-  </joint>
+  </joint> -->
   <!-- Top Link -->
-  <link name="${prefix}link2">
+  <!-- <link name="${prefix}link2">
     <collision>
       <origin xyz="0 0 ${height3/2 - axel_offset}" rpy="0 0 0"/>
@@ -101,13 +101,13 @@
         izz="${mass / 12.0 * (width*width + width*width)}"/>
     </inertial>
-  </link>
-  <joint name="${prefix}tool_joint" type="fixed">
+  </link> -->
+  <!-- <joint name="${prefix}tool_joint" type="fixed">
     <origin xyz="0 0 1" rpy="0 0 0" />
     <parent link="${prefix}link2"/>
     <child link="${prefix}tool_link" />
-  </joint>
+  </joint> -->
   <!-- Tool Link -->
-  <link name="${prefix}tool_link">
-  </link>
+  <!-- <link name="${prefix}tool_link">
+  </link> -->
   </xacro:macro>
 </robot>
