Commit message: funciona parcialmente la rueda

File: src/test2_ros2control/description/urdf/rrbot.urdf.xacro (robot description, xacro)
@@ -8,3 +8,6 @@
   <!-- Import RRBot ros2_control description -->
   <!-- <xacro:include filename="$(find test1_ros2control)/ros2_control/rrbot.ros2_control.xacro" /> -->
+  <xacro:rrbot prefix="$(arg prefix)">
+    <origin xyz="0 0 0" rpy="0 0 0" />
+  </xacro:rrbot>
 </robot>

File: src/test2_ros2control/description/urdf/rrbot_description.urdf.xacro (robot description, xacro)
@@ -1,46 +1,50 @@
 <?xml version="1.0"?>
 <robot xmlns:xacro="http://www.ros.org/wiki/xacro">
-  <!-- Definición de constantes para las dimensiones del robot -->
-  <xacro:property name="PI" value="3.1415926535897931"/>
-  <xacro:property name="base_mass" value="0.3" /> <!-- Masa base del robot -->
-  <xacro:property name="base_width" value="0.1" /> <!-- Ancho de la base del robot -->
-  <xacro:property name="base_length" value="0.1" /> <!-- Longitud de la base del robot -->
-  <xacro:property name="base_height" value="0.05" /> <!-- Altura de la base del robot -->
-  <xacro:property name="wheel_mass" value="0.3" /> <!-- Masa de las ruedas -->
-  <xacro:property name="wheel_len" value="0.020" /> <!-- Longitud de las ruedas -->
-  <xacro:property name="wheel_radius" value="0.015" /> <!-- Radio de las ruedas -->
-  <!-- Se define el enlace de la base del robot -->
-  <link name="${prefix}base_link" />
-  <!-- wheel Link -->
-  <link name="${prefix}wheel">
-    <collision>
-      <origin xyz="0 0 0" rpy="${PI/2} 0 0"/>
-      <geometry>
-        <cylinder length="${wheel_len}" radius="${wheel_radius}"/>
-      </geometry>
-    </collision>
-    <visual>
-      <origin xyz="0 0 0" rpy="${PI/2} 0 0"/>
-      <geometry>
-        <cylinder length="${wheel_len}" radius="${wheel_radius}"/>
-      </geometry>
-      <material name="black"/>
-    </visual>
-    <inertial>
-      <origin xyz="0 0 0" rpy="${PI/2} 0 0"/>
-      <mass value="${wheel_mass}"/>
-      <inertia
-        ixx="${wheel_mass / 12.0 * (3*wheel_radius*wheel_radius + wheel_len*wheel_len)}" ixy="0.0" ixz="0.0"
-        iyy="${wheel_mass / 12.0 * (3*wheel_radius*wheel_radius + wheel_len*wheel_len)}" iyz="0.0"
-        izz="${wheel_mass / 2.0 * wheel_radius*wheel_radius}"/>
-      </inertial>
+  <xacro:macro name="rrbot" params="prefix *origin">
+    <!-- Definición de constantes para las dimensiones del robot -->
+    <xacro:property name="PI" value="3.1415926535897931"/>
+    <xacro:property name="base_mass" value="0.3" /> <!-- Masa base del robot -->
+    <xacro:property name="base_width" value="0.1" /> <!-- Ancho de la base del robot -->
+    <xacro:property name="base_length" value="0.1" /> <!-- Longitud de la base del robot -->
+    <xacro:property name="base_height" value="0.05" /> <!-- Altura de la base del robot -->
+    <xacro:property name="wheel_mass" value="0.3" /> <!-- Masa de las ruedas -->
+    <xacro:property name="wheel_len" value="0.020" /> <!-- Longitud de las ruedas -->
+    <xacro:property name="wheel_radius" value="0.015" /> <!-- Radio de las ruedas -->
+    <xacro:property name="z_offset" value="-${base_height/2}" /> <!-- Desplazamiento vertical de la base del robot -->
+    <!-- Se define el enlace de la base del robot -->
+    <link name="${prefix}base_link">
     </link>
-  <joint name="${prefix}wheel_joint" type="continuous">
-    <parent link="${prefix}base_link"/>
-    <child link="${prefix}left_wheel"/>
-    <origin xyz="0 -${base_width/2} ${z_offset}" rpy="0 0 0"/>
-    <axis xyz="0 1 0"/>
-    <dynamics damping="0.2"/>
-    <limit effort="100" velocity="1.0"/>
-  </joint>
+    <joint name="${prefix}wheel_joint" type="continuous">
+      <parent link="${prefix}base_link"/>
+      <child link="${prefix}wheel"/>
+      <origin xyz="0 -${base_width/2} ${z_offset}" rpy="0 0 0"/>
+      <axis xyz="0 1 0"/>
+      <dynamics damping="0.2"/>
+      <limit effort="100" velocity="1.0"/>
+    </joint>
+    <!-- wheel Link -->
+    <link name="${prefix}wheel">
+      <collision>
+        <origin xyz="0 0 0" rpy="${PI/2} 0 0"/>
+        <geometry>
+          <cylinder length="${wheel_len}" radius="${wheel_radius}"/>
+        </geometry>
+      </collision>
+      <visual>
+        <origin xyz="0 0 0" rpy="${PI/2} 0 0"/>
+        <geometry>
+          <cylinder length="${wheel_len}" radius="${wheel_radius}"/>
+        </geometry>
+        <material name="black"/>
+      </visual>
+      <inertial>
+        <origin xyz="0 0 0" rpy="${PI/2} 0 0"/>
+        <mass value="${wheel_mass}"/>
+        <inertia
+          ixx="${wheel_mass / 12.0 * (3*wheel_radius*wheel_radius + wheel_len*wheel_len)}" ixy="0.0" ixz="0.0"
+          iyy="${wheel_mass / 12.0 * (3*wheel_radius*wheel_radius + wheel_len*wheel_len)}" iyz="0.0"
+          izz="${wheel_mass / 2.0 * wheel_radius*wheel_radius}"/>
+        </inertial>
+    </link>
+  </xacro:macro>
 </robot>

Commit message: se hace ajustes a propiedades de entrada inecesarios

File: src/test2_ros2control/description/urdf/rrbot.urdf.xacro (robot description, xacro)
@@ -8,8 +8,5 @@
   <!-- Import RRBot ros2_control description -->
   <xacro:include filename="$(find test2_ros2control)/ros2_control/rrbot.ros2_control.xacro" />
-  <xacro:rrbot prefix="$(arg prefix)">
-    <origin xyz="0 0 0" rpy="0 0 0" />
-  </xacro:rrbot>
-  <xacro:rrbot_ros2_control
-    name="RRBot" prefix="$(arg prefix)" />
+  <xacro:rrbot prefix="$(arg prefix)"/>
+  <xacro:rrbot_ros2_control name="RRBot" prefix="$(arg prefix)" />
 </robot>

File: src/test2_ros2control/description/urdf/rrbot_description.urdf.xacro (robot description, xacro)
@@ -1,5 +1,5 @@
 <?xml version="1.0"?>
 <robot xmlns:xacro="http://www.ros.org/wiki/xacro">
-  <xacro:macro name="rrbot" params="prefix *origin">
+  <xacro:macro name="rrbot" params="prefix">
     <!-- Definición de constantes para las dimensiones del robot -->
     <xacro:property name="PI" value="3.1415926535897931"/>
