Commit message: se corrigue los nombres de los joints

File: src/test2_ros2control/description/ros2_control/rrbot.ros2_control.xacro (robot description, xacro)
@@ -7,7 +7,7 @@
         <param name="hw_start_duration_sec">0</param>
         <param name="hw_stop_duration_sec">3.0</param>
-        <param name="hw_slowdown">100</param>
+        <param name="hw_slowdown">10</param>
       </hardware>
-      <joint name="${prefix}joint1">
+      <joint name="${prefix}wheel_joint">
         <command_interface name="position"/>
         <state_interface name="position"/>
